Commit message: initial gazebo state is done

File: my_robotarm_pkg/urdf/my_robotarm_gazebo_with_control_and_camera.xacro (robot description, xacro)
@@ -1,4 +1,5 @@
 <?xml version="1.0"?>
 <robot xmlns:xacro="http://www.ros.org/wiki/xacro" name="two_dof_robot">
+<xacro:include filename="$(find my_robotarm_pkg)/urdf/camera.xacro" />
   <!-- ==================== Global Material Definitions ==================== -->
   <material name="dark_grey">
@@ -172,3 +173,34 @@
     </plugin>
   </gazebo>
+  <!-- ROS 2 Control Hardware Interface -->
+  <ros2_control name="GazeboSimSystem" type="system">
+    <hardware>
+      <plugin>gz_ros2_control/GazeboSimSystem</plugin>
+    </hardware>
+    <joint name="joint1">
+      <command_interface name="position"/>
+      <state_interface name="position"/>
+      <state_interface name="velocity"/>
+    </joint>
+    <joint name="joint2">
+      <command_interface name="position"/>
+      <state_interface name="position"/>
+      <state_interface name="velocity"/>
+    </joint>
+    <joint name="right_finger_joint">
+      <command_interface name="position"/>
+      <state_interface name="position"/>
+      <state_interface name="velocity"/>
+    </joint>
+  </ros2_control>
+  <!-- Gazebo ROS 2 Control Plugin -->
+  <gazebo>
+    <plugin filename="gz_ros2_control-system" name="gz_ros2_control::GazeboSimROS2ControlPlugin">
+      <parameters>$(find my_robotarm_pkg)/config/controllers.yaml</parameters>
+    </plugin>
+  </gazebo>
+  <xacro:camera_sensor
+  parent_link="base_link"
+  x="0.20" y="0.0" z="0.25"
+  roll="0" pitch="0.5" yaw="3.14159" />
 </robot>
