Commit message: VM-host synch was out. Omit the prev commit. Now camera works intheworld

File: my_robotarm_pkg/urdf/camera.xacro (robot description, xacro)
@@ -42,4 +42,8 @@
         <visualize>true</visualize>
         <topic>camera/image_raw</topic>
+        <!-- URDF->SDF lumps the fixed camera joint into base_link, so the
+             default frame_id would be "two_dof_robot::base_link::camera",
+             which matches no TF frame. Force it to the URDF link name. -->
+        <gz_frame_id>camera_link</gz_frame_id>
         <camera>
           <camera_info_topic>camera/camera_info</camera_info_topic>

File: my_robotarm_pkg/urdf/my_robotarm_gazebo.xacro (robot description, xacro)
@@ -16,5 +16,10 @@
   </material>
   <!-- ==================== Links ==================== -->
-  <!-- Base Link (Fixed: Added inertial block so Gazebo keeps it) -->
+  <link name="world"/>
+  <joint name="world_to_base" type="fixed">
+    <parent link="world"/>
+    <child link="base_link"/>
+    <origin xyz="0 0 0" rpy="0 0 0"/>
+  </joint>
   <link name="base_link">
     <inertial>
@@ -196,10 +201,6 @@
   </gazebo>
   <xacro:camera_sensor
-    parent_link="base_link"
-    x="0.005"
-    y="0.0"
-    z="0.05"
-    roll="0"
-    pitch="0"
-    yaw="0" />
+  parent_link="base_link"
+  x="0.20" y="0.0" z="0.25"
+  roll="0" pitch="0.5" yaw="3.14159" />
 </robot>

File: my_robotarm_pkg/urdf/my_robotarm_with_ee.xacro (robot description, xacro)
@@ -2,5 +2,5 @@
 <robot name="two_dof_robot">
   <!-- Color Definitions -->
-  <material name="red">
+  <material name="dark_grey">
     <color rgba="0.2 0.2 0.2 1.0"/>
   </material>

Commit message: initial launch file notes are updated accordingly

File: my_robotarm_pkg/urdf/camera.xacro (robot description, xacro)
@@ -42,7 +42,4 @@
         <visualize>true</visualize>
         <topic>camera/image_raw</topic>
-        <!-- URDF->SDF lumps the fixed camera joint into base_link, so the
-             default frame_id would be "two_dof_robot::base_link::camera",
-             which matches no TF frame. Force it to the URDF link name. -->
         <gz_frame_id>camera_link</gz_frame_id>
         <camera>

File: my_robotarm_pkg/urdf/my_robotarm_gazebo.xacro (robot description, xacro)
@@ -1,4 +1,32 @@
 <?xml version="1.0"?>
 <robot xmlns:xacro="http://www.ros.org/wiki/xacro" name="two_dof_robot">
+<xacro:include filename="$(find my_robotarm_pkg)/urdf/camera.xacro" />
+<!-- ROS 2 Control Hardware Interface -->
+  <ros2_control name="GazeboSimSystem" type="system">
+    <hardware>
+      <plugin>gz_ros2_control/GazeboSimSystem</plugin>
+    </hardware>
+    <joint name="joint1">
+      <command_interface name="position"/>
+      <state_interface name="position"/>
+      <state_interface name="velocity"/>
+    </joint>
+    <joint name="joint2">
+      <command_interface name="position"/>
+      <state_interface name="position"/>
+      <state_interface name="velocity"/>
+    </joint>
+    <joint name="right_finger_joint">
+      <command_interface name="position"/>
+      <state_interface name="position"/>
+      <state_interface name="velocity"/>
+    </joint>
+  </ros2_control>
+  <!-- Gazebo ROS 2 Control Plugin -->
+  <gazebo>
+    <plugin filename="gz_ros2_control-system" name="gz_ros2_control::GazeboSimROS2ControlPlugin">
+      <parameters>$(find my_robotarm_pkg)/config/controllers.yaml</parameters>
+    </plugin>
+  </gazebo>
   <!-- ==================== Global Material Definitions ==================== -->
   <material name="dark_grey">
@@ -172,3 +200,7 @@
     </plugin>
   </gazebo>
+  <xacro:camera_sensor
+  parent_link="base_link"
+  x="0.20" y="0.0" z="0.25"
+  roll="0" pitch="0.5" yaw="3.14159" />
 </robot>
